File: Board.brd (EAGLE design)
At the start: 68.6 x 53.3 mm, 1 part

Commit message: Board is layed out
Parts:
- added POT_LEVER, POT_PUSH: (no value), con-lstb:MA03-1
- added YOKE1: (no value), con-lstb:MA07-1
- added YOKE2: (no value), con-lstb:MA12-1
Connections:
- new net S$1: E$1.5V, POT_LEVER.1, POT_PUSH.1, YOKE2.1
- new net S$10: E$1.D9, YOKE1.7
- new net S$11: E$1.A0, YOKE2.2
- new net S$12: E$1.A3, YOKE2.3
- new net S$13: E$1.D1, YOKE2.4
- new net S$14: E$1.D6, YOKE2.5
- new net S$15: E$1.A4, YOKE2.7
- new net S$16: E$1.A5, YOKE2.8
- new net S$17: E$1.D11, YOKE2.9
- new net S$18: E$1.D2, YOKE2.10
- new net S$19: E$1.D5, YOKE2.11
- new net S$2: E$1.GND1, E$1.GND2, POT_LEVER.3, POT_PUSH.3, YOKE2.12, YOKE2.6
- new net S$3: E$1.A1, POT_PUSH.2
- new net S$4: E$1.A2, POT_LEVER.2
- new net S$5: E$1.D3, YOKE1.2
- new net S$6: E$1.D4, YOKE1.3
- new net S$7: E$1.D7, YOKE1.4
- new net S$8: E$1.D8, YOKE1.5
- new net S$9: E$1.D10, YOKE1.6
Routing:
- net S$2: track 0.00 -> 66.1 mm
- net S$14: track 0.00 -> 57.6 mm
- net S$6: track 0.00 -> 57.5 mm
- net S$5: track 0.00 -> 55.3 mm
- net S$16: track 0.00 -> 55.0 mm
- net S$13: track 0.00 -> 52.3 mm
- net S$15: track 0.00 -> 51.8 mm
- net S$12: track 0.00 -> 49.5 mm
- net S$7: track 0.00 -> 45.4 mm
- net S$18: track 0.00 -> 44.4 mm
- net S$1: track 0.00 -> 41.9 mm
- net S$8: track 0.00 -> 39.0 mm
- net S$4: track 0.00 -> 38.2 mm
- net S$10: track 0.00 -> 35.0 mm
- net S$19: track 0.00 -> 34.1 mm
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