File: Board.brd (EAGLE design)
At the start: 68.6 x 53.3 mm, 6 parts

Commit message: Board is done
Parts:
- removed YOKE1: (no value), con-lstb:MA07-1
- removed YOKE2: (no value), con-lstb:MA12-1
- added POT_YOKE: (no value), adafruit:1X01
- added YOKE_1: (no value), pinhead:1X07
- added YOKE_2: (no value), pinhead:1X11
- RESET: device con-samtec:TSW-101-08-G-D -> pinhead:1X02
- moved RESET 8.03 mm to (6.35, 7.62), turned to 0 degrees
Connections:
- net S$3 renamed S$21
- removed net S$17: E$1.D11, YOKE2.9
- new net S$22: E$1.A2, POT_LEVER.2
- net S$1: now also E$1.D9, YOKE_1.7; no longer E$1.5V, POT_LEVER.1, POT_PUSH.1, YOKE2.1
- net S$10: now also E$1.D11, YOKE_2.9; no longer E$1.D9, YOKE1.7
- net S$11: now also E$1.A5, YOKE_2.8; no longer E$1.A0, YOKE2.2
- net S$12: now also E$1.A4, YOKE_2.7; no longer E$1.A3, YOKE2.3
- net S$13: now also E$1.D6, YOKE_2.5; no longer E$1.D1, YOKE2.4
- net S$14: now also E$1.D1, YOKE_2.4; no longer E$1.D6, YOKE2.5
- net S$15: now also E$1.A3, YOKE_2.3; no longer E$1.A4, YOKE2.7
- net S$16: now also E$1.A0, YOKE_2.2; no longer E$1.A5, YOKE2.8
- net S$18: now also E$1.RESET, RESET.1; no longer E$1.D2, YOKE2.10
- net S$19: now also E$1.5V, POT_LEVER.3, POT_PUSH.3, YOKE_2.1; no longer E$1.D5, YOKE2.11
- net S$2: now also E$1.D10, YOKE_1.6; no longer E$1.GND1, E$1.GND2, POT_LEVER.3, POT_PUSH.3, RESET.2, YOKE2.12, YOKE2.6
- net S$20: now also E$1.GND1, E$1.GND2, POT_LEVER.1, POT_PUSH.1, POT_YOKE.1, RESET.2, YOKE_2.6; no longer E$1.RESET, RESET.1
- net S$4: now also E$1.D8, YOKE_1.5; no longer E$1.A2, POT_LEVER.2
- net S$5: now also E$1.D7, YOKE_1.4; no longer E$1.D3, YOKE1.2
- net S$6: now also YOKE_1.3; no longer YOKE1.3
- net S$7: now also E$1.D3, YOKE_1.2; no longer E$1.D7, YOKE1.4
- net S$8: now also E$1.D5, YOKE_2.11; no longer E$1.D8, YOKE1.5
- net S$9: now also E$1.D2, YOKE_2.10; no longer E$1.D10, YOKE1.6
Routing:
- net S$20: track 21.0 -> 84.4 mm
- net S$2: track 86.8 -> 37.6 mm
- net S$22: track 0.00 -> 38.2 mm
- net S$19: track 34.1 -> 64.0 mm
- net S$17: track 27.2 -> 0.00 mm, vias 1 -> 0
- net S$11: track 33.8 -> 59.7 mm
- net S$7: track 45.4 -> 64.4 mm
- net S$16: track 55.0 -> 39.4 mm
- net S$9: track 31.8 -> 47.2 mm
- net S$18: track 44.4 -> 30.0 mm
- net S$13: track 52.3 -> 43.0 mm
- net S$10: track 35.0 -> 28.4 mm
- net S$12: track 49.5 -> 56.0 mm
- net S$5: track 55.3 -> 49.4 mm
- net S$4: track 38.2 -> 43.7 mm
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